Commit message: Add new data

File: model/resources/allegro_hand_description/urdf/allegro_arm.urdf (robot description, URDF)
Before this commit: robot allegro_arm, 26 links, 25 joints
Joints:
- joint joint_12: limit lower=0.263 upper=1.396 effort=15 velocity=7 -> lower=-0.11 upper=1.396 effort=15 velocity=7
- joint shoulder_0: origin xyz=-0.3 0.3 -0.5 rpy=0 0 0 -> xyz=0.5 0.0 0.2 rpy=0 2 3.1416

Commit message: interp is working add new data

File: model/resources/allegro_hand_description/urdf/allegro_arm.urdf (robot description, URDF)
Before this commit: robot allegro_arm, 26 links, 25 joints
Joints:
- joint elbow_1: limit lower=-2.00 upper=2.0 effort=15 velocity=7 -> lower=-2.0 upper=2.0 effort=15 velocity=7
- joint joint_0: limit lower=-0.47 upper=0.47 effort=15 velocity=7 -> lower=-0.6 upper=0.6 effort=15 velocity=7
- joint joint_1: limit lower=-0.196 upper=1.61 effort=15 velocity=7 -> lower=-0.5 upper=1.61 effort=15 velocity=7
- joint joint_12: limit lower=-0.11 upper=1.396 effort=15 velocity=7 -> lower=-0.2 upper=1.396 effort=15 velocity=7
- joint joint_4: limit lower=-0.47 upper=0.47 effort=15 velocity=7 -> lower=-0.6 upper=0.6 effort=15 velocity=7
- joint joint_5: limit lower=-0.196 upper=1.61 effort=15 velocity=7 -> lower=-0.5 upper=1.61 effort=15 velocity=7
- joint joint_8: limit lower=-0.47 upper=0.47 effort=15 velocity=7 -> lower=-0.6 upper=0.6 effort=15 velocity=7
- joint joint_9: limit lower=-0.196 upper=1.61 effort=15 velocity=7 -> lower=-0.5 upper=1.61 effort=15 velocity=7
- joint shoulder_0: origin xyz=0.5 0.0 0.2 rpy=0 2 3.1416 -> xyz=0.5 0.0 0.7 rpy=0 -2 0
- joint wrist_0: limit lower=-1.47 upper=1.47 effort=15 velocity=7 -> lower=-1.6 upper=1.6 effort=15 velocity=7
