Commit message: Add new gui interface for server

File: model/resources/allegro_hand_description/urdf/allegro_hand_description_right.urdf (robot description, URDF)
Before this commit: robot allegro_hand_right, 21 links, 20 joints
Links:
- removed link link_0.0
- removed link link_1.0
- removed link link_10.0
- removed link link_11.0
- removed link link_11.0_tip
- removed link link_12.0
- removed link link_13.0
- removed link link_14.0
- removed link link_15.0
- removed link link_15.0_tip
- removed link link_2.0
- removed link link_3.0
- removed link link_3.0_tip
- removed link link_4.0
- removed link link_5.0
- removed link link_6.0
- removed link link_7.0
- removed link link_7.0_tip
- removed link link_8.0
- removed link link_9.0
- added link hand_root
- added link link_0, mass 0.0119; collision box size=0.0196 0.0275 0.0164; visual mesh filename=../meshes/link_0.0.STL
- added link link_1, mass 0.065; collision box size=0.0196 0.0275 0.054; visual mesh filename=../meshes/link_1.0.STL
- added link link_10, mass 0.0355; collision box size=0.0196 0.0275 0.0384; visual mesh filename=../meshes/link_2.0.STL
- added link link_11, mass 0.0096; collision box size=0.0196 0.0275 0.0267; visual mesh filename=../meshes/link_3.0.STL
- added link link_11_tip, mass 0.0168; collision sphere radius=0.012; visual mesh filename=../meshes/link_3.0_tip.STL
- added link link_12, mass 0.0176; collision box size=0.0358 0.034 0.0455; visual mesh filename=../meshes/link_12.0_right.STL
- added link link_13, mass 0.0119; collision box size=0.0196 0.0275 0.0177; visual mesh filename=../meshes/link_13.0.STL
- added link link_14, mass 0.038; collision box size=0.0196 0.0275 0.0514; visual mesh filename=../meshes/link_14.0.STL
- added link link_15, mass 0.0388; collision box size=0.0196 0.0275 0.0423; visual mesh filename=../meshes/link_15.0.STL
- added link link_15_tip, mass 0.0168; collision sphere radius=0.012; visual mesh filename=../meshes/link_15.0_tip.STL
- added link link_2, mass 0.0355; collision box size=0.0196 0.0275 0.0384; visual mesh filename=../meshes/link_2.0.STL
- added link link_3, mass 0.0096; collision box size=0.0196 0.0275 0.0267; visual mesh filename=../meshes/link_3.0.STL
- added link link_3_tip, mass 0.0168; collision sphere radius=0.012; visual mesh filename=../meshes/link_3.0_tip.STL
- added link link_4, mass 0.0119; collision box size=0.0196 0.0275 0.0164; visual mesh filename=../meshes/link_0.0.STL
- added link link_5, mass 0.065; collision box size=0.0196 0.0275 0.054; visual mesh filename=../meshes/link_1.0.STL
- added link link_6, mass 0.0355; collision box size=0.0196 0.0275 0.0384; visual mesh filename=../meshes/link_2.0.STL
- added link link_7, mass 0.0096; collision box size=0.0196 0.0275 0.0267; visual mesh filename=../meshes/link_3.0.STL
- added link link_7_tip, mass 0.0168; collision sphere radius=0.012; visual mesh filename=../meshes/link_3.0_tip.STL
- added link link_8, mass 0.0119; collision box size=0.0196 0.0275 0.0164; visual mesh filename=../meshes/link_0.0.STL
- added link link_9, mass 0.065; collision box size=0.0196 0.0275 0.054; visual mesh filename=../meshes/link_1.0.STL
- link palm_link: geometry collision box size=0.0408 0.1130 0.095; visual mesh filename=../meshes/base_link.STL
Joints:
- removed joint joint_0.0
- removed joint joint_1.0
- removed joint joint_10.0
- removed joint joint_11.0
- removed joint joint_11.0_tip
- removed joint joint_12.0
- removed joint joint_13.0
- removed joint joint_14.0
- removed joint joint_15.0
- removed joint joint_15.0_tip
- removed joint joint_2.0
- removed joint joint_3.0
- removed joint joint_3.0_tip
- removed joint joint_4.0
- removed joint joint_5.0
- removed joint joint_6.0
- removed joint joint_7.0
- removed joint joint_7.0_tip
- removed joint joint_8.0
- removed joint joint_9.0
- added joint joint_0: type revolute, parent palm_link, child link_0, origin xyz=0 0.0435 -0.001542 rpy=-0.08726646255 0 0, axis 0 0 1, limit lower=-0.47 upper=0.47 effort=15 velocity=7
- added joint joint_1: type revolute, parent link_0, child link_1, origin xyz=0 0 0.0164, axis 0 1 0, limit lower=-0.196 upper=1.61 effort=15 velocity=7
- added joint joint_10: type revolute, parent link_9, child link_10, origin xyz=0 0 0.054, axis 0 1 0, limit lower=-0.174 upper=1.709 effort=15 velocity=7
- added joint joint_11: type revolute, parent link_10, child link_11, origin xyz=0 0 0.0384, axis 0 1 0, limit lower=-0.227 upper=1.618 effort=15 velocity=7
- added joint joint_11_tip: type fixed, parent link_11, child link_11_tip, origin xyz=0 0 0.0267 rpy=0 0 0
- added joint joint_12: type revolute, parent palm_link, child link_12, origin xyz=-0.0182 0.019333 -0.045987 rpy=0 -1.65806278845 -1.5707963259, axis -1 0 0, limit lower=0.263 upper=1.396 effort=15 velocity=7
- added joint joint_13: type revolute, parent link_12, child link_13, origin xyz=-0.027 0.005 0.0399, axis 0 0 1, limit lower=-0.105 upper=1.163 effort=15 velocity=7
- added joint joint_14: type revolute, parent link_13, child link_14, origin xyz=0 0 0.0177, axis 0 1 0, limit lower=-0.189 upper=1.644 effort=15 velocity=7
- added joint joint_15: type revolute, parent link_14, child link_15, origin xyz=0 0 0.0514, axis 0 1 0, limit lower=-0.162 upper=1.719 effort=15 velocity=7
- added joint joint_15_tip: type fixed, parent link_15, child link_15_tip, origin xyz=0 0 0.0423 rpy=0 0 0
- added joint joint_2: type revolute, parent link_1, child link_2, origin xyz=0 0 0.054, axis 0 1 0, limit lower=-0.174 upper=1.709 effort=15 velocity=7
- added joint joint_3: type revolute, parent link_2, child link_3, origin xyz=0 0 0.0384, axis 0 1 0, limit lower=-0.227 upper=1.618 effort=15 velocity=7
- added joint joint_3_tip: type fixed, parent link_3, child link_3_tip, origin xyz=0 0 0.0267 rpy=0 0 0
- added joint joint_4: type revolute, parent palm_link, child link_4, origin xyz=0 0 0.0007 rpy=0.0 0 0, axis 0 0 1, limit lower=-0.47 upper=0.47 effort=15 velocity=7
- added joint joint_5: type revolute, parent link_4, child link_5, origin xyz=0 0 0.0164, axis 0 1 0, limit lower=-0.196 upper=1.61 effort=15 velocity=7
- added joint joint_6: type revolute, parent link_5, child link_6, origin xyz=0 0 0.054, axis 0 1 0, limit lower=-0.174 upper=1.709 effort=15 velocity=7
- added joint joint_7: type revolute, parent link_6, child link_7, origin xyz=0 0 0.0384, axis 0 1 0, limit lower=-0.227 upper=1.618 effort=15 velocity=7
- added joint joint_7_tip: type fixed, parent link_7, child link_7_tip, origin xyz=0 0 0.0267 rpy=0 0 0
- added joint joint_8: type revolute, parent palm_link, child link_8, origin xyz=0 -0.0435 -0.001542 rpy=0.08726646255 0 0, axis 0 0 1, limit lower=-0.47 upper=0.47 effort=15 velocity=7
- added joint joint_9: type revolute, parent link_8, child link_9, origin xyz=0 0 0.0164, axis 0 1 0, limit lower=-0.196 upper=1.61 effort=15 velocity=7
- added joint root_to_base: type fixed, parent hand_root, child palm_link, origin xyz=0 0 0.095

Commit message: Add IK support for shadow hand

File: model/resources/allegro_hand_description/urdf/allegro_hand_description_right.urdf (robot description, URDF)
Before this commit: robot allegro_hand_right, 22 links, 21 joints
Links:
- link hand_root: mass None -> 1.0

File: model/resources/shadow_hand_description/urdf/shadow_hand_collision.urdf (robot description, URDF)
Before this commit: robot shadow_hand, 24 links, 23 joints
Links:
- link index_finger_distal: geometry collision capsule length=0.009 radius=0.008; visual capsule length=0.009 radius=0.008
- link index_finger_knuckle: geometry 
- link index_finger_middle: geometry collision capsule length=0.016 radius=0.008; visual capsule length=0.016 radius=0.008
- link index_finger_proximal: geometry collision capsule length=0.02 radius=0.009; visual capsule length=0.02 radius=0.009
- link little_finger_distal: geometry collision capsule length=0.009 radius=0.008; visual capsule length=0.009 radius=0.008
- link little_finger_knuckle: geometry 
- link little_finger_metacarpal: geometry 
- link little_finger_middle: geometry collision capsule length=0.016 radius=0.008; visual capsule length=0.016 radius=0.008
- link little_finger_proximal: geometry visual capsule length=0.01 radius=0.009
- link middle_finger_distal: geometry collision capsule length=0.009 radius=0.008; visual capsule length=0.009 radius=0.008
- link middle_finger_knuckle: geometry 
- link middle_finger_middle: geometry collision capsule length=0.017 radius=0.008; visual capsule length=0.017 radius=0.008
- link middle_finger_proximal: geometry collision capsule length=0.021 radius=0.009; visual capsule length=0.021 radius=0.009
- link palm: geometry collision box size=0.08 0.03 0.08; visual box size=0.08 0.03 0.08
- link ring_finger_distal: geometry collision capsule length=0.009 radius=0.008; visual capsule length=0.009 radius=0.008
- link ring_finger_knuckle: geometry 
- link ring_finger_middle: geometry collision capsule length=0.016 radius=0.008; visual capsule length=0.016 radius=0.008
- link ring_finger_proximal: geometry collision capsule length=0.01 radius=0.009; visual capsule length=0.01 radius=0.009
- link thumb_distal: geometry collision capsule length=0.012 radius=0.009; visual capsule length=0.012 radius=0.009
- link thumb_middle: geometry collision capsule length=0.01 radius=0.01; visual capsule length=0.01 radius=0.01
- link thumb_proximal: geometry 
