Commit message: Add simplified collision geometry for shadow hand

File: model/resources/shadow_hand_description/urdf/shadow_hand.urdf (robot description, URDF)
Before this commit: robot shadow_hand, 25 links, 24 joints
Links:
- removed link forearm
- removed link wrist
- link index_finger_distal: geometry collision capsule length=0.009 radius=0.008; visual mesh filename=shadow_hand/meshes/visual/finger_distal.dae
- link index_finger_knuckle: geometry visual mesh filename=shadow_hand/meshes/visual/knuckle.dae
- link index_finger_middle: geometry collision capsule length=0.016 radius=0.008; visual mesh filename=shadow_hand/meshes/visual/finger_middle.dae
- link index_finger_proximal: geometry collision capsule length=0.02 radius=0.009; visual mesh filename=shadow_hand/meshes/visual/finger_proximal.dae
- link little_finger_distal: geometry collision capsule length=0.009 radius=0.008; visual mesh filename=shadow_hand/meshes/visual/finger_distal.dae
- link little_finger_knuckle: geometry visual mesh filename=shadow_hand/meshes/visual/knuckle.dae
- link little_finger_metacarpal: geometry visual mesh filename=shadow_hand/meshes/visual/metacarpal.dae
- link little_finger_middle: geometry collision capsule length=0.016 radius=0.008; visual mesh filename=shadow_hand/meshes/visual/finger_middle.dae
- link little_finger_proximal: geometry collision capsule length=0.02 radius=0.009; visual mesh filename=shadow_hand/meshes/visual/finger_proximal.dae
- link middle_finger_distal: geometry collision capsule length=0.009 radius=0.008; visual mesh filename=shadow_hand/meshes/visual/finger_distal.dae
- link middle_finger_knuckle: geometry visual mesh filename=shadow_hand/meshes/visual/knuckle.dae
- link middle_finger_middle: geometry collision capsule length=0.017 radius=0.008; visual mesh filename=shadow_hand/meshes/visual/finger_middle.dae
- link middle_finger_proximal: geometry collision capsule length=0.021 radius=0.009; visual mesh filename=shadow_hand/meshes/visual/finger_proximal.dae
- link palm: geometry collision box size=0.08 0.03 0.08; visual mesh filename=shadow_hand/meshes/visual/palm.dae
- link ring_finger_distal: geometry collision capsule length=0.009 radius=0.008; visual mesh filename=shadow_hand/meshes/visual/finger_distal.dae
- link ring_finger_knuckle: geometry visual mesh filename=shadow_hand/meshes/visual/knuckle.dae
- link ring_finger_middle: geometry collision capsule length=0.016 radius=0.008; visual mesh filename=shadow_hand/meshes/visual/finger_middle.dae
- link ring_finger_proximal: geometry collision capsule length=0.02 radius=0.009; visual mesh filename=shadow_hand/meshes/visual/finger_proximal.dae
- link thumb_distal: geometry collision capsule length=0.012 radius=0.009; visual mesh filename=shadow_hand/meshes/visual/thumb_distal.dae
- link thumb_middle: geometry collision capsule length=0.02 radius=0.01; visual mesh filename=shadow_hand/meshes/visual/thumb_middle.dae
- link thumb_proximal: geometry collision capsule length=0.015 radius=0.012; visual mesh filename=shadow_hand/meshes/visual/thumb_proximal.dae
Joints:
- removed joint forearm_joint
- removed joint wrist_joint
