Commit message: Add new demo

File: envs/assets/cardboard.urdf (robot description, URDF)
Before this commit: robot pen, 1 links, 0 joints
Links:
- removed link penBody
- added link cardboardBody, mass 1.0; collision box size=0.4 0.4 0.002; visual box size=0.4 0.4 0.002

File: envs/assets/ruler.urdf (robot description, URDF)
Before this commit: robot pen, 1 links, 0 joints
Links:
- removed link penBody
- added link rulerBody, mass 1.0; collision box size=0.36 0.028 0.002; visual mesh filename=ruler.obj scale=2 2 2

File: envs/assets/ruler_collision.urdf (robot description, URDF)
Before this commit: robot pen, 1 links, 0 joints
Links:
- removed link penBody
- added link rulerBody, mass 1.0; collision box size=0.36 0.014 0.002; visual box size=0.36 0.028 0.002
