Commit message: sync

File: envs/assets/box.urdf (robot description, URDF)
Before this commit: robot box, 1 links, 0 joints
Links:
- link boxLink: geometry collision mesh filename=box.stl scale=1 1 0.8; visual mesh filename=box.stl scale=1 1 0.8

File: envs/assets/cardboard.urdf (robot description, URDF)
Before this commit: robot cardboard, 1 links, 0 joints
Links:
- link cardboardBody: mass 1.0 -> 2.0; geometry collision box size=0.24 0.4 0.002; visual mesh filename=box.stl scale=0.6 1 0.02

File: envs/assets/pen.urdf (robot description, URDF)
Before this commit: robot pen, 1 links, 0 joints
Links:
- link penBody: mass 1.0 -> 2.0

File: envs/assets/plate_cvx_simple.urdf (robot description, URDF)
Before this commit: robot plate_cvx_simple, 1 links, 0 joints
Links:
- link plateLink: mass 1.0 -> 4.0

File: envs/assets/ruler.urdf (robot description, URDF)
Before this commit: robot ruler, 1 links, 0 joints
Links:
- link rulerBody: mass 1.0 -> 2.0; geometry collision box size=0.36 0.028 0.002; visual mesh filename=ruler.obj scale=1 1 1
