Commit message: upload ablation

File: envs/assets/book.urdf (robot description, URDF)
Before this commit: robot book, 1 links, 0 joints
Links:
- link boxLink: geometry collision box size=0.4 0.4 0.015; visual mesh filename=book.obj scale=1 1 0.3

File: envs/assets/keyboard.urdf (robot description, URDF)
Before this commit: robot laptop, 1 links, 0 joints
Links:
- link boxLink: mass 1.0 -> 3.0

Commit message: release

File: envs/assets/book.urdf (robot description, URDF)
Before this commit: robot book, 1 links, 0 joints
Links:
- link boxLink: geometry collision box size=0.4 0.4 0.05; visual mesh filename=book.obj scale=1 1 1
